Commit message: build .urdf file to check

File: src/hrwros_support/urdf/hrwros.urdf (robot description, URDF)
Before this commit: robot hrwros, 29 links, 29 joints
Links:
- removed link robot2_base
- removed link robot2_base_link
- removed link robot2_ee_link
- removed link robot2_forearm_link
- removed link robot2_pedestal_link
- removed link robot2_shoulder_link
- removed link robot2_tool0
- removed link robot2_upper_arm_link
- removed link robot2_wrist_1_link
- removed link robot2_wrist_2_link
- removed link robot2_wrist_3_link
Joints:
- removed joint robot2-robot2_pedestal_joint
- removed joint robot2_base_link-base_fixed_joint
- removed joint robot2_ee_fixed_joint
- removed joint robot2_elbow_joint
- removed joint robot2_pedestal_joint
- removed joint robot2_shoulder_lift_joint
- removed joint robot2_shoulder_pan_joint
- removed joint robot2_wrist_1_joint
- removed joint robot2_wrist_2_joint
- removed joint robot2_wrist_3_joint
- removed joint robot2_wrist_3_link-tool0_fixed_joint
- joint bin_1_joint: origin xyz=-8.0 -2.2 0 rpy=0 0 0 -> xyz=-0.3 1.2 0.0 rpy=0 0 0

Commit message: add basic form of pedestal in urdf

File: src/hrwros_support/urdf/hrwros.urdf (robot description, URDF)
Before this commit: robot hrwros, 18 links, 18 joints
Links:
- added link robot2_pedestal_link; visual box size=1 1 1
Joints:
- added joint robot2_pedestal_joint: type fixed, parent world, child robot2_pedestal_link
- joint bin_1_joint: origin xyz=-0.3 1.2 0.0 rpy=0 0 0 -> xyz=-8.3 -2.2 0.0 rpy=0 0 0

File: src/hrwros_support/urdf/hrwros.xacro (robot description, xacro)
@@ -48,3 +48,14 @@
     <origin xyz="-8.3 -2.2 0.0" rpy="0 0 0" />
   </joint>
+  <link name="robot2_pedestal_link">
+    <visual>
+     <geometry>
+       <box size="1 1 1" />
+     </geometry>
+    </visual>
+  </link>
+  <joint name="robot2_pedestal_joint" type="fixed">
+    <parent link="world" />
+    <child link="robot2_pedestal_link" />
+  </joint>
 </robot>
