Commit message: remove bin 2,3,4 from urdf

File: src/hrwros_support/urdf/hrwros.xacro (robot description, xacro)
@@ -20,8 +20,4 @@
   <xacro:include filename="$(find hrwros_support)/urdf/bin/bin.urdf.xacro"/>
   <xacro:bin_urdf prefix="bin_1_"/>
-  <xacro:bin_urdf prefix="bin_2_"/>
-  <xacro:bin_urdf prefix="bin_3_"/>
-  <xacro:bin_urdf prefix="bin_4_"/>
-  <xacro:bin_urdf prefix="bin_5_"/>
   <!-- Joints -->
   <joint name="world_interface_to_world" type="fixed">
@@ -52,27 +48,3 @@
     <origin xyz="-0.3 1.2 0.0" rpy="0 0 0" />
   </joint>
-  <!-- bin 2 -->
-  <joint name="bin_2_joint" type="fixed">
-    <parent link="world_interface" />
-    <child link="bin_2_base_link" />
-    <origin xyz="-0.3 0.4 0.0" rpy="0 0 0" />
-  </joint>
-  <!-- bin 3 -->
-  <joint name="bin_3_joint" type="fixed">
-    <parent link="world_interface" />
-    <child link="bin_3_base_link" />
-    <origin xyz="-0.3 -0.4 0.0" rpy="0 0 0" />
-  </joint>
-  <!-- bin 4 -->
-  <joint name="bin_4_joint" type="fixed">
-    <parent link="world_interface" />
-    <child link="bin_4_base_link" />
-    <origin xyz="-0.3 -1.2 0.0" rpy="0 0 0" />
-  </joint>
-  <!-- bin 5 -->
-  <joint name="bin_5_joint" type="fixed">
-    <parent link="world_interface" />
-    <child link="bin_5_base_link" />
-    <origin xyz="-0.3 -2.0 0.0" rpy="0 0 0" />
-  </joint>
 </robot>

Commit message: move bin near pallet boxs

File: src/hrwros_support/urdf/hrwros.xacro (robot description, xacro)
@@ -46,5 +46,5 @@
     <parent link="world_interface" />
     <child link="bin_1_base_link" />
-    <origin xyz="-0.3 1.2 0.0" rpy="0 0 0" />
+    <origin xyz="-8.3 -2.2 0.0" rpy="0 0 0" />
   </joint>
 </robot>

Commit message: revise dimenstion of pedestal in urdf

File: src/hrwros_support/urdf/hrwros.xacro (robot description, xacro)
@@ -50,6 +50,7 @@
   <link name="robot2_pedestal_link">
     <visual>
+     <origin xyz="0 0 0.3"/>
      <geometry>
-       <box size="1 1 1" />
+       <box size="0.3 0.3 0.6" />
      </geometry>
     </visual>

Commit message: change color of pedestal to blue color in hrwros.xacro

File: src/hrwros_support/urdf/hrwros.xacro (robot description, xacro)
@@ -54,4 +54,7 @@
        <box size="0.3 0.3 0.6" />
      </geometry>
+     <material name="robot2_pedestal_colour">
+      <color rgba="0 0.16 0.53 1"/>
+     </material>
     </visual>
   </link>

Commit message: move pedestal next to boxs and left of bin

File: src/hrwros_support/urdf/hrwros.xacro (robot description, xacro)
@@ -62,4 +62,5 @@
     <parent link="world" />
     <child link="robot2_pedestal_link" />
+    <origin xyz="-7.8 -1.5 0"/>
   </joint>
 </robot>

Commit message: corrected bin pos from x -8.3 to 8

File: src/hrwros_support/urdf/hrwros.xacro (robot description, xacro)
@@ -46,5 +46,5 @@
     <parent link="world_interface" />
     <child link="bin_1_base_link" />
-    <origin xyz="-8.3 -2.2 0.0" rpy="0 0 0" />
+    <origin xyz="-8 -2.2 0.0" rpy="0 0 0" />
   </joint>
   <link name="robot2_pedestal_link">

Commit message: add ur5 robot on top of pedestal in hrwros.xacro

File: src/hrwros_support/urdf/hrwros.xacro (robot description, xacro)
@@ -64,3 +64,10 @@
     <origin xyz="-7.8 -1.5 0"/>
   </joint>
+  <xacro:include filename="$(find ur_description)/urdf/ur5.urdf.xacro"/>
+  <xacro:ur5_robot prefix="robot2_" joint_limited="true"/>
+  <joint name="robot2-robot2_pedestal_joint" type="fixed">
+   <parent link="robot2_pedestal_link"/>
+   <child link="robot2_base_link" />
+   <origin xyz="0 0 0.6" rpy="0 0 ${radians(90)}"/>
+  </joint>
 </robot>

Commit message: add second bin opposite to robot1 seperated by conveyour 2.1 x for origin

File: src/hrwros_support/urdf/hrwros.xacro (robot description, xacro)
@@ -20,4 +20,5 @@
   <xacro:include filename="$(find hrwros_support)/urdf/bin/bin.urdf.xacro"/>
   <xacro:bin_urdf prefix="bin_1_"/>
+  <xacro:bin_urdf prefix="bin_2_"/>
   <!-- Joints -->
   <joint name="world_interface_to_world" type="fixed">
@@ -48,4 +49,10 @@
     <origin xyz="-8 -2.2 0.0" rpy="0 0 0" />
   </joint>
+   <!-- bin 2 -->
+  <joint name="bin_2_joint" type="fixed">
+    <parent link="world_interface" />
+    <child link="bin_2_base_link" />
+    <origin xyz="2.1 1.8 0.0" rpy="0 0 0" />
+  </joint>
   <link name="robot2_pedestal_link">
     <visual>

Commit message: Add green sphere of 40cm radius beneath stairs in urfd

File: src/hrwros_support/urdf/hrwros.xacro (robot description, xacro)
@@ -78,3 +78,19 @@
    <origin xyz="0 0 0.6" rpy="0 0 ${radians(90)}"/>
   </joint>
+   <link name="sphere_link">
+     <visual>
+       <origin xyz="0 0 0.2"/>
+       <geometry>
+        <sphere radius="0.2" />
+       </geometry>
+       <material name="sphere_colour">
+         <color rgba="0.1 1 0.1 1"/>
+       </material>
+      </visual>
+    </link>
+ <joint name="sphere_world_joint" type="fixed">
+    <parent link="world" />
+    <child link="sphere_link" />
+    <origin xyz="5.8 -5.5 0"/>
+  </joint>
 </robot>

Commit message: Week 3 Setup Done

File: src/hrwros_support/urdf/hrwros.xacro (robot description, xacro)
@@ -17,7 +17,31 @@
   <xacro:include filename="$(find hrwros_support)/urdf/vacuum_gripper/vacuum_gripper.urdf.xacro"/>
   <xacro:vacuum_gripper_urdf prefix="vacuum_gripper1_" joint_prefix="vacuum_gripper1_joint"/>
+  <!-- Robot2 Pedestal -->
+  <xacro:include filename="$(find hrwros_support)/urdf/robot_pedestal/robot_pedestal.urdf.xacro"/>
+  <xacro:robot_pedestal_urdf pedestal_prefix="robot2_" pedestal_parent="world_interface" pedestal_height="0.7">
+    <origin xyz="-7.8 -1.5 0.0" rpy="0 0 0"/>
+  </xacro:robot_pedestal_urdf>
+  <!-- Robot2 -->
+  <xacro:include filename="$(find ur_description)/urdf/ur5.urdf.xacro"/>
+  <xacro:ur5_robot prefix="robot2_" joint_limited="true"/>
+  <!-- Vacuum Gripper2 -->
+  <xacro:include filename="$(find hrwros_support)/urdf/vacuum_gripper/vacuum_gripper.urdf.xacro"/>
+  <xacro:vacuum_gripper_urdf prefix="vacuum_gripper2_" joint_prefix="vacuum_gripper2_joint"/>
   <!-- bins -->
   <xacro:include filename="$(find hrwros_support)/urdf/bin/bin.urdf.xacro"/>
   <xacro:bin_urdf prefix="bin_1_"/>
+  <!-- logical camera 1 collision model -->
+  <xacro:include filename="$(find hrwros_support)/urdf/logical_camera/logical_camera.urdf.xacro"/>
+  <xacro:logical_camera_urdf prefix="logical_camera1_" logical_camera_parent="world_interface">
+    <origin xyz="1.2 1.8 2.0" rpy="0 1.5708 0"/>
+  </xacro:logical_camera_urdf>
+  <!-- logical camera 2 collision model -->
+  <xacro:include filename="$(find hrwros_support)/urdf/logical_camera/logical_camera.urdf.xacro"/>
+  <xacro:logical_camera_urdf prefix="logical_camera2_" logical_camera_parent="world_interface">
+    <origin xyz="-8.3 -1.23 1.8" rpy="0 1.5708 0"/>
+  </xacro:logical_camera_urdf>
+  <!-- break beam -->
+  <xacro:include filename="$(find hrwros_support)/urdf/break_beam/break_beam.urdf.xacro"/>
+  <xacro:break_beam_urdf prefix="break_beam_"/>
   <!-- Joints -->
   <joint name="world_interface_to_world" type="fixed">
@@ -33,6 +57,6 @@
   <!-- robot1 to pedestal. -->
   <joint name="robot1_to_pedestal" type="fixed">
-  <origin xyz="0 0 0.95" rpy="0 0 0" />
-  <parent link="robot1_pedestal_link" />
+  <origin xyz="0.5 1.8 0.95" rpy="0 0 0" />
+  <parent link="world_interface" />
   <child link="robot1_base_link" />
   </joint>
@@ -42,32 +66,31 @@
     <child link="vacuum_gripper1_base_link" />
   </joint>
-  <!-- bin 1 -->
+  <!-- robot2-pedestal to world. -->
+  <joint name="robot2_pedestal_to_world_interface" type="fixed">
+    <parent link="world_interface" />
+    <child link="robot2_pedestal_link" />
+    <origin xyz="-7.8 -1.5 0.0" rpy="0.0 0.0 0.0"/>
+  </joint>
+  <!-- robot2 to pedestal. -->
+  <joint name="robot2_to_pedestal" type="fixed">
+    <parent link="world_interface" />
+    <child link="robot2_base_link" />
+    <origin xyz="-7.8 -1.5 0.7" rpy="0 0 1.57" />
+  </joint>
+  <!-- gripper2 to robot2. -->
+  <joint name="gripper2_to_robot2" type="fixed">
+    <parent link="robot2_tool0" />
+    <child link="vacuum_gripper2_base_link" />
+  </joint>
+  <!-- break beam to world. -->
+  <joint name="break_beam_joint" type="fixed">
+    <parent link="world_interface" />
+    <child link="break_beam_world_interface" />
+  </joint>
+  <!-- bin to world. -->
   <joint name="bin_1_joint" type="fixed">
     <parent link="world_interface" />
     <child link="bin_1_base_link" />
-    <origin xyz="-8 -2.2 0.0" rpy="0 0 0" />
-  </joint>
-  <link name="robot2_pedestal_link">
-    <visual>
-     <origin xyz="0 0 0.3"/>
-     <geometry>
-       <box size="0.3 0.3 0.6" />
-     </geometry>
-     <material name="robot2_pedestal_colour">
-      <color rgba="0 0.16 0.53 1"/>
-     </material>
-    </visual>
-  </link>
-  <joint name="robot2_pedestal_joint" type="fixed">
-    <parent link="world" />
-    <child link="robot2_pedestal_link" />
-    <origin xyz="-7.8 -1.5 0"/>
-  </joint>
-  <xacro:include filename="$(find ur_description)/urdf/ur5.urdf.xacro"/>
-  <xacro:ur5_robot prefix="robot2_" joint_limited="true"/>
-  <joint name="robot2-robot2_pedestal_joint" type="fixed">
-   <parent link="robot2_pedestal_link"/>
-   <child link="robot2_base_link" />
-   <origin xyz="0 0 0.6" rpy="0 0 ${radians(90)}"/>
+    <origin xyz="-8.0 -2.2 0.0" rpy="0 0 0" />
   </joint>
 </robot>

File: src/hrwros_support/urdf/robot_system/robot_system.gazebo.xacro (robot description, xacro)
@@ -1,10 +1,19 @@
 <?xml version="1.0"?>
 <robot name="robot_system" xmlns:xacro="http://www.ros.org/wiki/xacro">
-  <xacro:macro name="robot_system_gazebo" params="robot_prefix robot_parameter_name">
+  <xacro:macro name="robot_system_gazebo" params="robot_prefix robot_parameter_name vacuum_gripper_prefix gripper_plugin_name">
     <!-- Vacuum Gripper -->
-    <!-- <xacro:include filename="$(find hrwros_support)/urdf/vacuum_gripper/vacuum_gripper.gazebo.xacro"/>
-    <xacro:vacuum_gripper_gazebo prefix="${vacuum_gripper_prefix}" gripper_link="robot_system_::robot_wrist_3_link">
-      <drops_info/>
-    </xacro:vacuum_gripper_gazebo> -->
+    <xacro:if value="${robot_prefix == 'robot1_'}">
+      <xacro:include filename="$(find hrwros_support)/urdf/vacuum_gripper/vacuum_gripper.gazebo.xacro"/>
+      <xacro:vacuum_gripper_gazebo prefix="${vacuum_gripper_prefix}" gripper_link="robot1::${robot_prefix}wrist_3_link" plugin_name = "${gripper_plugin_name}">
+        <drops_info/>
+      </xacro:vacuum_gripper_gazebo>
+    </xacro:if>
+    <xacro:if value="${robot_prefix == 'robot2_'}">
+      <xacro:include filename="$(find hrwros_support)/urdf/vacuum_gripper/vacuum_gripper.gazebo.xacro"/>
+      <xacro:vacuum_gripper_gazebo prefix="${vacuum_gripper_prefix}" gripper_link="robot2::${robot_prefix}wrist_3_link" plugin_name = "${gripper_plugin_name}">
+        <drops_info/>
+      </xacro:vacuum_gripper_gazebo>
+    </xacro:if>
+<!--
     <gazebo reference="${robot_prefix}base_link">
       <turnGravityOff>true</turnGravityOff>
@@ -28,4 +37,11 @@
       <turnGravityOff>true</turnGravityOff>
     </gazebo>
+    <gazebo reference="${robot_prefix}ee_link">
+      <turnGravityOff>true</turnGravityOff>
+    </gazebo>
+    <gazebo reference="${vacuum_gripper_prefix}suction_cup">
+      <turnGravityOff>true</turnGravityOff>
+    </gazebo>
+-->
     <gazebo>
       <plugin name="gazebo_ros_control" filename="libgazebo_ros_control.so">

File: src/hrwros_support/urdf/robot_system/robot_system.urdf.xacro (robot description, xacro)
@@ -2,12 +2,17 @@
 <robot name="robot_system" xmlns:xacro="http://www.ros.org/wiki/xacro">
   <xacro:macro name="robot_system_urdf" params="robot_prefix vacuum_gripper_prefix robot_type">
+  <xacro:arg name="transmission_hw_interface" default="hardware_interface/EffortJointInterface" />
+    <!-- Used for fixing robot to Gazebo 'base_link' -->
+    <link name="world"/>
     <!-- Robot -->
     <xacro:if value="${robot_type == 'ur10'}">
       <xacro:include filename="$(find ur_description)/urdf/ur10.urdf.xacro"/>
-      <xacro:ur10_robot prefix="${robot_prefix}" joint_limited="true"/>
+      <xacro:ur10_robot prefix="${robot_prefix}" joint_limited="true"
+        transmission_hw_interface="$(arg transmission_hw_interface)"/>
     </xacro:if>
     <xacro:if value="${robot_type == 'ur5'}">
       <xacro:include filename="$(find ur_description)/urdf/ur5.urdf.xacro"/>
-      <xacro:ur5_robot prefix="${robot_prefix}" joint_limited="true"/>
+      <xacro:ur5_robot prefix="${robot_prefix}" joint_limited="true"
+           transmission_hw_interface="$(arg transmission_hw_interface)"/>
     </xacro:if>
     <!-- Vacuum Gripper -->
@@ -19,4 +24,10 @@
       <child link="${vacuum_gripper_prefix}base_link" />
     </joint>
+    <!-- joint list -->
+    <joint name="${robot_prefix}world_joint" type="fixed">
+      <parent link="world" />
+      <child link="${robot_prefix}base_link" />
+      <!-- <origin xyz="0.8 1.8 0.95" rpy="0 0 0" />-->
+    </joint>
 </xacro:macro>
 </robot>

File: src/hrwros_support/urdf/robot_system/robot_system.xacro (robot description, xacro)
@@ -5,10 +5,10 @@
   <xacro:arg name="vacuum_gripper_prefix" default="vacuum_gripper1_"/>
   <xacro:arg name="robot_param" default="/robot1/robot1_description"/>
+  <xacro:arg name="gripper_plugin_name" default="gripper1"/>
   <!-- URDF -->
   <xacro:include filename="$(find hrwros_support)/urdf/robot_system/robot_system.urdf.xacro"/>
-  <xacro:robot_system_urdf robot_type= "$(arg robot_type)" robot_prefix="$(arg robot_prefix)" vacuum_gripper_prefix="$(arg vacuum_gripper_prefix"/>
+  <xacro:robot_system_urdf robot_type= "$(arg robot_type)" robot_prefix="$(arg robot_prefix)" vacuum_gripper_prefix="$(arg vacuum_gripper_prefix)"/>
   <!-- Gazebo -->
   <xacro:include filename="$(find hrwros_support)/urdf/robot_system/robot_system.gazebo.xacro"/>
-  <xacro:robot_system_gazebo robot_prefix="$(arg robot_prefix)" robot_parameter_name="$(arg robot_param)"/>
-  <!-- <xacro:robot_system_gazebo parent_link_linear_actuator="$(arg parent_linear_actuator)"/> -->
+  <xacro:robot_system_gazebo robot_prefix="$(arg robot_prefix)" robot_parameter_name="$(arg robot_param)" vacuum_gripper_prefix="$(arg vacuum_gripper_prefix)" gripper_plugin_name="$(arg gripper_plugin_name)"/>
 </robot>
